File: relay.kicad_pcb (KiCad board)
At the start: 2 copper layers, 167.6 x 77.5 mm, 92 parts, among them J1 TAP, J10 PGH, J11 PGH, J2 TBP, J3 PTA, J4 PTB, J5 PGH, J6 Jack-DC, J7 TO_FTDI, J8 P, J9 PGH, K1 G5LE-1, K2 G5LE-1, K3 G5LE-1, K4 G5LE-1, K5 G5LE-1, K6 G5LE-1, K7 G5LE-1, K8 G5LE-1, K9 G5LE-1, Q1 BC847, Q2 BC847, Q3 BC847, Q4 BC847, Q5 BC847, Q6 BC847, Q7 BC847, Q8 BC847, Q9 BC847, SW1 Button, SW2 Button, U1 PC817, U10 PC817, U11 PC817, U12 74HC595, U2 PC817, U3 PC817, U4 PC817, U5 PC817, U6 ESP-12E, U7 PC817, U8 AMS1117-3.3, U9 PC817

Commit message: ready
Parts:
- moved J7 3.81 mm to (45.7, 82.5), turned to -90 degrees
- moved R20 3.81 mm to (144.8, 59.7)
- moved R19 3.29 mm to (144.8, 63.5)
- moved NT1 1.31 mm to (79.9, 83.8), turned to 0 degrees
- moved R11 1.27 mm to (115.1, 86.9)
- moved R12 1.27 mm to (111.8, 86.9)
- moved U10 1.27 mm to (161.3, 53.3)
- turned D13 to 90 degrees
Routing:
- net VCC: track 0.00 -> 701.4 mm, vias 0 -> 2
- net /VIN: track 0.00 -> 401.7 mm, vias 0 -> 2
- net /TB_P: track 0.00 -> 151.6 mm, vias 0 -> 2
- net /P_TA: track 0.00 -> 138.9 mm, vias 0 -> 2
- net /TA_P: track 0.00 -> 102.7 mm, vias 0 -> 2
- net /P_GH: track 0.00 -> 86.9 mm, vias 0 -> 2
- net GND: track 0.00 -> 80.2 mm, vias 0 -> 6
- net /Pompa: track 0.00 -> 68.6 mm, vias 0 -> 2
- net /P_SB: track 0.00 -> 68.2 mm, vias 0 -> 2
- net /TX: track 0.00 -> 62.1 mm
- net /RX: track 0.00 -> 58.1 mm
- net /P_TB: track 0.00 -> 57.2 mm, vias 0 -> 4
- net /RESET: track 0.00 -> 51.6 mm
- net /P_SC: track 0.00 -> 49.8 mm, vias 0 -> 2
- net /P_SA: track 0.00 -> 47.1 mm, vias 0 -> 2
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- added copper zone on B.Cu, net GND
- added copper zone on F.Cu, net GND
Other:
- outline, holes or cut-outs redrawn
